File: zynq/DRAM_sch.kicad_sch (KiCad schematic)
At the start: 1 part, among them IC2 MT41J128M16JT-125_K

Commit message: .
Connections:
- net DDR_D13: now reaches IC2.A2 (DQ13)
- net DDR_D15: now reaches IC2.A3 (DQ15)
- net DDR_D12: now reaches IC2.A7 (DQ12)
- net DDR_DQS1_N: now reaches IC2.B7 (UDQS#)
- net DDR_D14: now reaches IC2.B8 (DQ14)
- net DDR_D11: now reaches IC2.C2 (DQ11)
- net DDR_D9: now reaches IC2.C3 (DQ9)
- net DDR_DQS1_P: now reaches IC2.C7 (UDQS)
- net DDR_D10: now reaches IC2.C8 (DQ10)
- net DDR_DM1: now reaches IC2.D3 (UDM)
- net DDR_D8: now reaches IC2.D7 (DQ8)
- net DDR_D0: now reaches IC2.E3 (DQ0)
- net DDR_DM0: now reaches IC2.E7 (LDM)
- net DDR_D2: now reaches IC2.F2 (DQ2)
- net DDR_DQS0_P: now reaches IC2.F3 (LDQS)
- net DDR_D1: now reaches IC2.F7 (DQ1)
- net DDR_D3: now reaches IC2.F8 (DQ3)
- net DDR_D6: now reaches IC2.G2 (DQ6)
- net DDR_DQS0_N: now reaches IC2.G3 (LDQS#)
- net DDR_D4: now reaches IC2.H3 (DQ4)
- net DDR_D7: now reaches IC2.H7 (DQ7)
- net DDR_D5: now reaches IC2.H8 (DQ5)
- net DDR_RAS: now reaches IC2.J3 (RAS#)
- net DDR_CK_P: now reaches IC2.J7 (CK)
- net DDR_ODT0: now reaches IC2.K1 (ODT)
- net DDR_CAS: now reaches IC2.K3 (CAS#)
- net DDR_CK_N: now reaches IC2.K7 (CK#)
- net DDR_CKE0: now reaches IC2.K9 (CKE)
- net DDR_CS: now reaches IC2.L2 (CS#)
- net DDR_WE: now reaches IC2.L3 (WE#)
- net DDR_BA0: now reaches IC2.M2 (BA0)
- net DDR_BA2: now reaches IC2.M3 (BA2)
- net DDR_BA1: now reaches IC2.N8 (BA1)
- net DDR_RESET: now reaches IC2.T2 (RESET#)

Commit message: .
Changed lines of the file:
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@@
     (effects (font (size 1.27 1.27)) (justify left bottom))
   )
-  (label "DDR3_CS" (at 88.9 69.85 0)
+  (label "DDR_CS" (at 88.9 69.85 0)
     (effects (font (size 1.27 1.27)) (justify left bottom))
   )
@@
     (effects (font (size 1.27 1.27)) (justify left bottom))
   )
-  (label "DDR3_RAS" (at 88.9 41.91 0)
+  (label "DDR_RAS" (at 88.9 41.91 0)
     (effects (font (size 1.27 1.27)) (justify left bottom))
   )
@@
     (effects (font (size 1.27 1.27)) (justify left bottom))
   )
-  (label "DDR3_CAS" (at 119.38 152.4 0)
+  (label "DDR_CAS" (at 119.38 152.4 0)
     (effects (font (size 1.27 1.27)) (justify left bottom))
   )
@@
     (effects (font (size 1.27 1.27)) (justify left bottom))
   )
-  (label "DDR3_CS" (at 119.38 144.78 0)
+  (label "DDR_CS" (at 119.38 144.78 0)
     (effects (font (size 1.27 1.27)) (justify left bottom))
   )
@@
     (effects (font (size 1.27 1.27)) (justify left bottom))
   )
-  (label "DDR3_WE" (at 119.38 156.21 0)
+  (label "DDR_WE" (at 119.38 156.21 0)
     (effects (font (size 1.27 1.27)) (justify left bottom))
   )
@@
     (effects (font (size 1.27 1.27)) (justify left bottom))
   )
-  (label "DDR3_CAS" (at 88.9 57.15 0)
+  (label "DDR_CAS" (at 88.9 57.15 0)
     (effects (font (size 1.27 1.27)) (justify left bottom))
   )
@@
     (effects (font (size 1.27 1.27)) (justify left bottom))
   )
-  (label "DDR3_RAS" (at 119.38 148.59 0)
+  (label "DDR_RAS" (at 119.38 148.59 0)
     (effects (font (size 1.27 1.27)) (justify left bottom))
   )
@@
     (effects (font (size 1.27 1.27)) (justify left bottom))
   )
-  (label "DDR3_WE" (at 88.9 72.39 0)
+  (label "DDR_WE" (at 88.9 72.39 0)
     (effects (font (size 1.27 1.27)) (justify left bottom))
   )
