File: zynq/POWER_sch.kicad_sch (KiCad schematic)
At the start: 1 part, among them J1 POWER_SOURCE

Commit message: .
Parts:
- removed J1: POWER_SOURCE, Connector_PinHeader_2.54mm:PinHeader_1x06_P2.54mm_Vertical, symbol Connector:Conn_01x06_Male
Other:
- note removed: "(notes) POWER SUPPLY 3.3V --> 1.5A 1.8V --> 0.6A 1.5V --> 1.2A 1.0V --> 2.1A"
Changed lines of the file:
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@@
 (kicad_sch (version 20211123) (generator eeschema)
   (paper "A4")
-  (bus (pts (xy 86.36 44.45) (xy 97.79 44.45))
-    (stroke (width 0) (type default) (color 0 0 0 0))
-  )
-  (bus (pts (xy 86.36 36.83) (xy 97.79 36.83))
-    (stroke (width 0) (type default) (color 0 0 0 0))
-  )
-  (bus (pts (xy 86.36 39.37) (xy 97.79 39.37))
-    (stroke (width 0) (type default) (color 0 0 0 0))
-  )
-  (bus (pts (xy 86.36 46.99) (xy 97.79 46.99))
-    (stroke (width 0) (type default) (color 0 0 0 0))
-  )
-  (bus (pts (xy 86.36 41.91) (xy 97.79 41.91))
-    (stroke (width 0) (type default) (color 0 0 0 0))
-  )
-  (bus (pts (xy 86.36 49.53) (xy 97.79 49.53))
-    (stroke (width 0) (type default) (color 0 0 0 0))
-  )
-  (text "(notes) POWER SUPPLY\n\n3.3V --> 1.5A\n1.8V --> 0.6A\n1.5V --> 1.2A\n1.0V --> 2.1A"
-    (at 130.81 45.72 0)
-    (effects (font (size 1.27 1.27) italic) (justify right bottom))
-  )
-  (global_label "1.8V" (shape input) (at 97.79 41.91 0) (fields_autoplaced)
-    (effects (font (size 1.27 1.27)) (justify left))
-    (property "Intersheet References" "${INTERSHEET_REFS}" (id 0) (at 104.3155 41.8306 0)
-      (effects (font (size 1.27 1.27)) (justify left) hide)
-    )
-  )
-  (global_label "1.5V" (shape input) (at 97.79 44.45 0) (fields_autoplaced)
-    (effects (font (size 1.27 1.27)) (justify left))
-    (property "Intersheet References" "${INTERSHEET_REFS}" (id 0) (at 104.3155 44.3706 0)
-      (effects (font (size 1.27 1.27)) (justify left) hide)
-    )
-  )
-  (global_label "1.0V" (shape input) (at 97.79 46.99 0) (fields_autoplaced)
-    (effects (font (size 1.27 1.27)) (justify left))
-    (property "Intersheet References" "${INTERSHEET_REFS}" (id 0) (at 104.3155 46.9106 0)
-      (effects (font (size 1.27 1.27)) (justify left) hide)
-    )
-  )
-  (global_label "3.3V" (shape input) (at 97.79 39.37 0) (fields_autoplaced)
-    (effects (font (size 1.27 1.27)) (justify left))
-    (property "Intersheet References" "${INTERSHEET_REFS}" (id 0) (at 104.3155 39.2906 0)
-      (effects (font (size 1.27 1.27)) (justify left) hide)
-    )
-  )
-  (global_label "5V" (shape input) (at 97.79 36.83 0) (fields_autoplaced)
-    (effects (font (size 1.27 1.27)) (justify left))
-    (property "Intersheet References" "${INTERSHEET_REFS}" (id 0) (at 102.5012 36.7506 0)
-      (effects (font (size 1.27 1.27)) (justify left) hide)
-    )
-  )
-  (global_label "GND" (shape input) (at 97.79 49.53 0) (fields_autoplaced)
-    (effects (font (size 1.27 1.27)) (justify left))
-    (property "Intersheet References" "${INTERSHEET_REFS}" (id 0) (at 104.0736 49.4506 0)
-      (effects (font (size 1.27 1.27)) (justify left) hide)
-    )
-  )
-  (symbol (lib_id "Connector:Conn_01x06_Male") (at 81.28 41.91 0) (unit 1)
-    (in_bom yes) (on_board yes) (fields_autoplaced)
-    (property "Reference" "J1" (id 0) (at 81.915 31.75 0))
-    (property "Value" "POWER_SOURCE" (id 1) (at 81.915 34.29 0))
-    (property "Footprint" "Connector_PinHeader_2.54mm:PinHeader_1x06_P2.54mm_Vertical" (id 2) (at 81.28 41.91 0)
-      (effects (font (size 1.27 1.27)) hide)
-    )
-    (property "Datasheet" "~" (id 3) (at 81.28 41.91 0)
-      (effects (font (size 1.27 1.27)) hide)
-    )
-    (pin "1")
-    (pin "2")
-    (pin "3")
-    (pin "4")
-    (pin "5")
-    (pin "6")
-  )
 )
