File: zynq/XC7Z010_sch.kicad_sch (KiCad schematic)
At the start: 1 part

Commit message: .
Connections:
- net DDR3_D13: now reaches IC1.A2 (PS_DDR_DQ2_502)
- net DDR3_D15: now reaches IC1.A4 (PS_DDR_DQ3_502)
- net DDR3_D12: now reaches IC1.B3 (PS_DDR_DQ1_502)
- net DDR3_D10: now reaches IC1.C1 (PS_DDR_DQ6_502)
- net DDR3_D11: now reaches IC1.C3 (PS_DDR_DQ0_502)
- net DDR3_D14: now reaches IC1.D1 (PS_DDR_DQ5_502)
- net DDR3_D8: now reaches IC1.D3 (PS_DDR_DQ4_502)
- net DDR3_D9: now reaches IC1.E1 (PS_DDR_DQ7_502)
- net DDR3_D2: now reaches IC1.E2 (PS_DDR_DQ8_502)
- net DDR3_D0: now reaches IC1.E3 (PS_DDR_DQ9_502)
- net DDR3_D3: now reaches IC1.G3 (PS_DDR_DQ10_502)
- net DDR3_D7: now reaches IC1.H1 (PS_DDR_DQ14_502)
- net DDR3_D1: now reaches IC1.H2 (PS_DDR_DQ13_502)
- net DDR3_D5: now reaches IC1.H3 (PS_DDR_DQ11_502)
- net DDR3_D4: now reaches IC1.J1 (PS_DDR_DQ15_502)
- net DDR3_D6: now reaches IC1.J3 (PS_DDR_DQ12_502)
- net DDR3_BA2: now reaches IC1.J5 (PS_DDR_BA2_502)
- net DDR3_CK_P: now reaches IC1.L2 (PS_DDR_CKP_502)
- net DDR3_BA0: now reaches IC1.L5 (PS_DDR_BA0_502)
- net DDR3_CK_N: now reaches IC1.M2 (PS_DDR_CKN_502)
- net DDR3_CKE0: now reaches IC1.N3 (PS_DDR_CKE_502)
- net DDR3_BA1: now reaches IC1.R4 (PS_DDR_BA1_502)

Commit message: .
Connections:
- net DDR3_CAS: now also IC1.P5 (PS_DDR_CAS_B_502)
- net DDR3_CS: now also IC1.N1 (PS_DDR_CS_B_502)
- net DDR3_DM0: now also IC1.F1 (PS_DDR_DM1_502)
- net DDR3_DM1: now also IC1.A1 (PS_DDR_DM0_502)
- net DDR3_DQS0_N: now also IC1.F2 (PS_DDR_DQS_N1_502)
- net DDR3_DQS0_P: now also IC1.G2 (PS_DDR_DQS_P1_502)
- net DDR3_DQS1_N: now also IC1.B2 (PS_DDR_DQS_N0_502)
- net DDR3_DQS1_P: now also IC1.C2 (PS_DDR_DQS_P0_502)
- net DDR3_ODT0: now also IC1.N5 (PS_DDR_ODT_502)
- net DDR3_RAS: now also IC1.P4 (PS_DDR_RAS_B_502)
- net DDR3_RESET: now also IC1.B4 (PS_DDR_DRST_B_502)
- net DDR3_WE: now also IC1.M5 (PS_DDR_WE_B_502)
Changed lines of the file:
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@@
+    (stroke (width 0) (type default) (color 0 0 0 0))
+  )
+  (wire (pts (xy 83.82 147.32) (xy 100.33 147.32))
     (stroke (width 0) (type default) (color 0 0 0 0))
   )
@@
     (stroke (width 0) (type default) (color 0 0 0 0))
   )
+  (wire (pts (xy 176.53 154.94) (xy 193.04 154.94))
+    (stroke (width 0) (type default) (color 0 0 0 0))
+  )
   (wire (pts (xy 83.82 200.66) (xy 100.33 200.66))
     (stroke (width 0) (type default) (color 0 0 0 0))
@@
     (stroke (width 0) (type default) (color 0 0 0 0))
   )
+  (wire (pts (xy 83.82 297.18) (xy 100.33 297.18))
+    (stroke (width 0) (type default) (color 0 0 0 0))
+  )
   (bus (pts (xy 337.82 76.2) (xy 337.82 80.01))
     (stroke (width 0) (type default) (color 0 0 0 0))
@@
     (stroke (width 0) (type default) (color 0 0 0 0))
   )
+  (wire (pts (xy 83.82 299.72) (xy 100.33 299.72))
+    (stroke (width 0) (type default) (color 0 0 0 0))
+  )
   (wire (pts (xy 83.82 50.8) (xy 100.33 50.8))
     (stroke (width 0) (type default) (color 0 0 0 0))
@@
     (stroke (width 0) (type default) (color 0 0 0 0))
   )
+  (wire (pts (xy 176.53 144.78) (xy 193.04 144.78))
+    (stroke (width 0) (type default) (color 0 0 0 0))
+  )
   (wire (pts (xy 83.82 195.58) (xy 100.33 195.58))
     (stroke (width 0) (type default) (color 0 0 0 0))
@@
     (stroke (width 0) (type default) (color 0 0 0 0))
   )
+  (wire (pts (xy 83.82 350.52) (xy 100.33 350.52))
+    (stroke (width 0) (type default) (color 0 0 0 0))
+  )
   (wire (pts (xy 83.82 45.72) (xy 100.33 45.72))
     (stroke (width 0) (type default) (color 0 0 0 0))
@@
     (stroke (width 0) (type default) (color 0 0 0 0))
   )
+  (wire (pts (xy 83.82 96.52) (xy 100.33 96.52))
+    (stroke (width 0) (type default) (color 0 0 0 0))
+  )
   (bus (pts (xy 337.82 68.58) (xy 337.82 72.39))
     (stroke (width 0) (type default) (color 0 0 0 0))
   )
+  (wire (pts (xy 176.53 203.2) (xy 193.04 203.2))
+    (stroke (width 0) (type default) (color 0 0 0 0))
+  )
   (wire (pts (xy 83.82 401.32) (xy 100.33 401.32))
     (stroke (width 0) (type default) (color 0 0 0 0))
@@
     (stroke (width 0) (type default) (color 0 0 0 0))
   )
+  (wire (pts (xy 176.53 104.14) (xy 193.04 104.14))
+    (stroke (width 0) (type default) (color 0 0 0 0))
+  )
   (wire (pts (xy 83.82 505.46) (xy 100.33 505.46))
     (stroke (width 0) (type default) (color 0 0 0 0))
@@
     (stroke (width 0) (type default) (color 0 0 0 0))
   )
+  (wire (pts (xy 176.53 205.74) (xy 193.04 205.74))
+    (stroke (width 0) (type default) (color 0 0 0 0))
+  )
   (wire (pts (xy 455.93 67.31) (xy 445.77 67.31))
     (stroke (width 0) (type default) (color 0 0 0 0))
@@
     (stroke (width 0) (type default) (color 0 0 0 0))
   )
+  (wire (pts (xy 83.82 43.18) (xy 100.33 43.18))
+    (stroke (width 0) (type default) (color 0 0 0 0))
+  )
   (bus (pts (xy 443.23 49.53) (xy 443.23 53.34))
     (stroke (width 0) (type default) (color 0 0 0 0))
@@
     (stroke (width 0) (type default) (color 0 0 0 0))
   )
+  (wire (pts (xy 83.82 101.6) (xy 100.33 101.6))
+    (stroke (width 0) (type default) (color 0 0 0 0))
+  )
   (wire (pts (xy 455.93 78.74) (xy 445.77 78.74))
     (stroke (width 0) (type default) (color 0 0 0 0))
@@
     (effects (font (size 1.27 1.27)) (justify left bottom))
   )
+  (label "DDR3_DQS1_P" (at 86.36 147.32 0)
+    (effects (font (size 1.27 1.27)) (justify left bottom))
+  )
   (label "DDR3_A8" (at 88.9 500.38 0)
     (effects (font (size 1.27 1.27)) (justify left bottom))
   )
+  (label "DDR3_RESET" (at 85.09 101.6 0)
+    (effects (font (size 1.27 1.27)) (justify left bottom))
+  )
   (label "DDR3_A0" (at 181.61 147.32 0)
     (effects (font (size 1.27 1.27)) (justify left bottom))
@@
     (effects (font (size 1.27 1.27)) (justify left bottom))
   )
+  (label "DDR3_RAS" (at 180.34 203.2 0)
+    (effects (font (size 1.27 1.27)) (justify left bottom))
+  )
   (label "DDR3_D0" (at 447.04 44.45 0)
     (effects (font (size 1.27 1.27)) (justify left bottom))
@@
     (effects (font (size 1.27 1.27)) (justify left bottom))
   )
-  (label "DDR3_DQS0_P" (at 284.48 54.61 0)
+  (label "DDR3_DQS0_P" (at 283.21 54.61 0)
     (effects (font (size 1.27 1.27)) (justify left bottom))
   )
@@
     (effects (font (size 1.27 1.27)) (justify left bottom))
   )
+  (label "DDR3_CS" (at 181.61 144.78 0)
+    (effects (font (size 1.27 1.27)) (justify left bottom))
+  )
   (label "DDR3_CAS" (at 242.57 74.93 0)
     (effects (font (size 1.27 1.27)) (justify left bottom))
@@
     (effects (font (size 1.27 1.27)) (justify left bottom))
   )
-  (label "DDR3_DQS0_N" (at 284.48 58.42 0)
+  (label "DDR3_DQS0_N" (at 283.21 58.42 0)
     (effects (font (size 1.27 1.27)) (justify left bottom))
   )
@@
     (effects (font (size 1.27 1.27)) (justify left bottom))
   )
+  (label "DDR3_DQS0_N" (at 85.09 299.72 0)
+    (effects (font (size 1.27 1.27)) (justify left bottom))
+  )
   (label "DDR3_D12" (at 447.04 90.17 0)
     (effects (font (size 1.27 1.27)) (justify left bottom))
@@
     (effects (font (size 1.27 1.27)) (justify left bottom))
   )
-  (label "DDR3_DQS1_P" (at 284.48 46.99 0)
+  (label "DDR3_DQS1_P" (at 283.21 46.99 0)
+    (effects (font (size 1.27 1.27)) (justify left bottom))
+  )
+  (label "DDR3_CAS" (at 180.34 205.74 0)
     (effects (font (size 1.27 1.27)) (justify left bottom))
   )
@@
     (effects (font (size 1.27 1.27)) (justify left bottom))
   )
+  (label "DDR3_DM1" (at 87.63 43.18 0)
+    (effects (font (size 1.27 1.27)) (justify left bottom))
+  )
   (label "DDR3_A6" (at 181.61 50.8 0)
     (effects (font (size 1.27 1.27)) (justify left bottom))
@@
     (effects (font (size 1.27 1.27)) (justify left bottom))
   )
+  (label "DDR3_DM0" (at 85.09 297.18 0)
+    (effects (font (size 1.27 1.27)) (justify left bottom))
+  )
   (label "DDR3_D15" (at 447.04 101.6 0)
     (effects (font (size 1.27 1.27)) (justify left bottom))
@@
     (effects (font (size 1.27 1.27)) (justify left bottom))
   )
-  (label "DDR3_DQS1_N" (at 284.48 50.8 0)
+  (label "DDR3_DQS1_N" (at 283.21 50.8 0)
+    (effects (font (size 1.27 1.27)) (justify left bottom))
+  )
+  (label "DDR3_WE" (at 181.61 104.14 0)
+    (effects (font (size 1.27 1.27)) (justify left bottom))
+  )
+  (label "DDR3_DQS1_N" (at 85.09 96.52 0)
     (effects (font (size 1.27 1.27)) (justify left bottom))
   )
@@
     (effects (font (size 1.27 1.27)) (justify left bottom))
   )
+  (label "DDR3_ODT0" (at 181.61 154.94 0)
+    (effects (font (size 1.27 1.27)) (justify left bottom))
+  )
   (label "DDR3_D11" (at 87.63 149.86 0)
     (effects (font (size 1.27 1.27)) (justify left bottom))
   )
+  (label "DDR3_DQS0_P" (at 86.36 350.52 0)
+    (effects (font (size 1.27 1.27)) (justify left bottom))
+  )
