File: zynq/zynq.kicad_sch (KiCad schematic)
At the start: 1 part

Commit message: .
Parts:
- removed IC1: (no value), symbol XC7Z010-1CLG400C:XC7Z010-1CLG400C
Other:
- added sheet CPU (XC7Z010_sch.kicad_sch)
- added sheet DRAM (DRAM_sch.kicad_sch)
- added sheet POWER_SUPPLY (POWER_sch.kicad_sch)

Commit message: .
Other:
- sheet DRAM renamed DDR3
- sheet CPU ports: added DDR3_BA[0..2], DDR3_CAS, DDR3_CKE0, DDR3_CK_N, DDR3_CK_P, DDR3_CS, DDR3_DM0, DDR3_DM1, DDR3_DQS0_N, DDR3_DQS0_P, DDR3_DQS1_N, DDR3_DQS1_P, DDR3_D[0..15], DDR3_ODT0, DDR3_RAS, DDR3_RESET, DDR3_WE; removed none
- sheet DDR3 ports: added DDR_BA[0..2], DDR_CAS, DDR_CKE0, DDR_CK_N, DDR_CK_P, DDR_CS, DDR_DM0, DDR_DM1, DDR_DQS0_N, DDR_DQS0_P, DDR_DQS1_N, DDR_DQS1_P, DDR_D[0..15], DDR_ODT0, DDR_RAS, DDR_RESET, DDR_WE; removed none
Changed lines of the file:
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@@
     (title "ZYNQ")
   )
-  (bus (pts (xy 93.98 97.79) (xy 115.57 97.79))
+  (bus (pts (xy 96.52 105.41) (xy 115.57 105.41))
     (stroke (width 0) (type default) (color 0 0 0 0))
   )
-  (sheet (at 58.42 88.9) (size 35.56 30.48) (fields_autoplaced)
+  (wire (pts (xy 96.52 125.73) (xy 115.57 125.73))
+    (stroke (width 0) (type default) (color 0 0 0 0))
+  )
+  (wire (pts (xy 96.52 152.4) (xy 115.57 152.4))
+    (stroke (width 0) (type default) (color 0 0 0 0))
+  )
+  (wire (pts (xy 96.52 128.27) (xy 115.57 128.27))
+    (stroke (width 0) (type default) (color 0 0 0 0))
+  )
+  (wire (pts (xy 96.52 161.29) (xy 115.57 161.29))
+    (stroke (width 0) (type default) (color 0 0 0 0))
+  )
+  (bus (pts (xy 96.52 97.79) (xy 115.57 97.79))
+    (stroke (width 0) (type default) (color 0 0 0 0))
+  )
+  (wire (pts (xy 96.52 135.89) (xy 115.57 135.89))
+    (stroke (width 0) (type default) (color 0 0 0 0))
+  )
+  (wire (pts (xy 96.52 147.32) (xy 115.57 147.32))
+    (stroke (width 0) (type default) (color 0 0 0 0))
+  )
+  (bus (pts (xy 96.52 101.6) (xy 115.57 101.6))
+    (stroke (width 0) (type default) (color 0 0 0 0))
+  )
+  (wire (pts (xy 96.52 138.43) (xy 115.57 138.43))
+    (stroke (width 0) (type default) (color 0 0 0 0))
+  )
+  (wire (pts (xy 96.52 149.86) (xy 115.57 149.86))
+    (stroke (width 0) (type default) (color 0 0 0 0))
+  )
+  (wire (pts (xy 96.52 154.94) (xy 115.57 154.94))
+    (stroke (width 0) (type default) (color 0 0 0 0))
+  )
+  (wire (pts (xy 96.52 120.65) (xy 115.57 120.65))
+    (stroke (width 0) (type default) (color 0 0 0 0))
+  )
+  (wire (pts (xy 96.52 166.37) (xy 115.57 166.37))
+    (stroke (width 0) (type default) (color 0 0 0 0))
+  )
+  (wire (pts (xy 96.52 140.97) (xy 115.57 140.97))
+    (stroke (width 0) (type default) (color 0 0 0 0))
+  )
+  (wire (pts (xy 96.52 118.11) (xy 115.57 118.11))
+    (stroke (width 0) (type default) (color 0 0 0 0))
+  )
+  (wire (pts (xy 96.52 115.57) (xy 115.57 115.57))
+    (stroke (width 0) (type default) (color 0 0 0 0))
+  )
+  (wire (pts (xy 96.52 133.35) (xy 115.57 133.35))
+    (stroke (width 0) (type default) (color 0 0 0 0))
+  )
+  (sheet (at 58.42 88.9) (size 38.1 81.28) (fields_autoplaced)
     (stroke (width 0.1524) (type solid) (color 0 0 0 0))
     (fill (color 0 0 0 0.0000))
@@
       (effects (font (size 1.27 1.27)) (justify left bottom))
     )
-    (property "Sheet file" "XC7Z010_sch.kicad_sch" (id 1) (at 58.42 119.9646 0)
+    (property "Sheet file" "XC7Z010_sch.kicad_sch" (id 1) (at 58.42 170.7646 0)
       (effects (font (size 1.27 1.27)) (justify left top))
     )
-    (pin "DDR3_A[0..14]" output (at 93.98 97.79 0)
+    (pin "DDR3_A[0..14]" output (at 96.52 97.79 0)
+      (effects (font (size 1.27 1.27)) (justify right))
+    )
+    (pin "DDR3_BA[0..2]" output (at 96.52 105.41 0)
+      (effects (font (size 1.27 1.27)) (justify right))
+    )
+    (pin "DDR3_CK_P" output (at 96.52 115.57 0)
+      (effects (font (size 1.27 1.27)) (justify right))
+    )
+    (pin "DDR3_CK_N" output (at 96.52 118.11 0)
+      (effects (font (size 1.27 1.27)) (justify right))
+    )
+    (pin "DDR3_CKE0" output (at 96.52 120.65 0)
+      (effects (font (size 1.27 1.27)) (justify right))
+    )
+    (pin "DDR3_D[0..15]" bidirectional (at 96.52 101.6 0)
+      (effects (font (size 1.27 1.27)) (justify right))
+    )
+    (pin "DDR3_ODT0" input (at 96.52 161.29 0)
+      (effects (font (size 1.27 1.27)) (justify right))
+    )
+    (pin "DDR3_DQS0_N" input (at 96.52 140.97 0)
+      (effects (font (size 1.27 1.27)) (justify right))
+    )
+    (pin "DDR3_RESET" input (at 96.52 166.37 0)
+      (effects (font (size 1.27 1.27)) (justify right))
+    )
+    (pin "DDR3_DM0" input (at 96.52 125.73 0)
+      (effects (font (size 1.27 1.27)) (justify right))
+    )
+    (pin "DDR3_DQS1_P" input (at 96.52 133.35 0)
+      (effects (font (size 1.27 1.27)) (justify right))
+    )
+    (pin "DDR3_DM1" input (at 96.52 128.27 0)
+      (effects (font (size 1.27 1.27)) (justify right))
+    )
+    (pin "DDR3_DQS1_N" input (at 96.52 135.89 0)
+      (effects (font (size 1.27 1.27)) (justify right))
+    )
+    (pin "DDR3_DQS0_P" input (at 96.52 138.43 0)
+      (effects (font (size 1.27 1.27)) (justify right))
+    )
+    (pin "DDR3_RAS" input (at 96.52 147.32 0)
+      (effects (font (size 1.27 1.27)) (justify right))
+    )
+    (pin "DDR3_CS" input (at 96.52 149.86 0)
+      (effects (font (size 1.27 1.27)) (justify right))
+    )
+    (pin "DDR3_WE" input (at 96.52 154.94 0)
+      (effects (font (size 1.27 1.27)) (justify right))
+    )
+    (pin "DDR3_CAS" input (at 96.52 152.4 0)
       (effects (font (size 1.27 1.27)) (justify right))
     )
   )
-  (sheet (at 115.57 88.9) (size 39.37 30.48) (fields_autoplaced)
+  (sheet (at 115.57 88.9) (size 39.37 81.28) (fields_autoplaced)
     (stroke (width 0.1524) (type solid) (color 0 0 0 0))
     (fill (color 0 0 0 0.0000))
-    (property "Sheet name" "DRAM" (id 0) (at 115.57 88.1884 0)
+    (property "Sheet name" "DDR3" (id 0) (at 115.57 88.1884 0)
       (effects (font (size 1.27 1.27)) (justify left bottom))
     )
-    (property "Sheet file" "DRAM_sch.kicad_sch" (id 1) (at 115.57 119.9646 0)
+    (property "Sheet file" "DRAM_sch.kicad_sch" (id 1) (at 115.57 170.7646 0)
       (effects (font (size 1.27 1.27)) (justify left top))
     )
@@
       (effects (font (size 1.27 1.27)) (justify left))
     )
+    (pin "DDR_CK_P" input (at 115.57 115.57 180)
+      (effects (font (size 1.27 1.27)) (justify left))
+    )
+    (pin "DDR_CKE0" input (at 115.57 120.65 180)
+      (effects (font (size 1.27 1.27)) (justify left))
+    )
+    (pin "DDR_CK_N" input (at 115.57 118.11 180)
+      (effects (font (size 1.27 1.27)) (justify left))
+    )
+    (pin "DDR_D[0..15]" bidirectional (at 115.57 101.6 180)
+      (effects (font (size 1.27 1.27)) (justify left))
+    )
+    (pin "DDR_BA[0..2]" input (at 115.57 105.41 180)
+      (effects (font (size 1.27 1.27)) (justify left))
+    )
+    (pin "DDR_DM0" input (at 115.57 125.73 180)
+      (effects (font (size 1.27 1.27)) (justify left))
+    )
+    (pin "DDR_DM1" input (at 115.57 128.27 180)
+      (effects (font (size 1.27 1.27)) (justify left))
+    )
+    (pin "DDR_ODT0" input (at 115.57 161.29 180)
+      (effects (font (size 1.27 1.27)) (justify left))
+    )
+    (pin "DDR_RESET" input (at 115.57 166.37 180)
+      (effects (font (size 1.27 1.27)) (justify left))
+    )
+    (pin "DDR_DQS1_N" input (at 115.57 135.89 180)
+      (effects (font (size 1.27 1.27)) (justify left))
+    )
+    (pin "DDR_DQS0_P" input (at 115.57 138.43 180)
+      (effects (font (size 1.27 1.27)) (justify left))
+    )
+    (pin "DDR_DQS0_N" input (at 115.57 140.97 180)
+      (effects (font (size 1.27 1.27)) (justify left))
+    )
+    (pin "DDR_DQS1_P" input (at 115.57 133.35 180)
+      (effects (font (size 1.27 1.27)) (justify left))
+    )
+    (pin "DDR_RAS" input (at 115.57 147.32 180)
+      (effects (font (size 1.27 1.27)) (justify left))
+    )
+    (pin "DDR_CS" input (at 115.57 149.86 180)
+      (effects (font (size 1.27 1.27)) (justify left))
+    )
+    (pin "DDR_CAS" input (at 115.57 152.4 180)
+      (effects (font (size 1.27 1.27)) (justify left))
+    )
+    (pin "DDR_WE" input (at 115.57 154.94 180)
+      (effects (font (size 1.27 1.27)) (justify left))
+    )

Commit message: .
Parts:
- added J?: POWER_SOURCE, Connector_PinHeader_2.54mm:PinHeader_1x06_P2.54mm_Vertical, symbol Connector:Conn_01x06_Male
Other:
- removed sheet POWER_SUPPLY
- note added: "(notes) POWER SUPPLY 3.3V --> 1.5A 1.8V --> 0.6A 1.5V --> 1.2A 1.0V --> 2.1A"
Changed lines of the file:
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@@
+    (stroke (width 0) (type default) (color 0 0 0 0))
+  )
+  (bus (pts (xy 35.56 30.48) (xy 46.99 30.48))
+    (stroke (width 0) (type default) (color 0 0 0 0))
+  )
+  (bus (pts (xy 35.56 38.1) (xy 46.99 38.1))
     (stroke (width 0) (type default) (color 0 0 0 0))
   )
@@
     (stroke (width 0) (type default) (color 0 0 0 0))
   )
+  (bus (pts (xy 35.56 25.4) (xy 46.99 25.4))
+    (stroke (width 0) (type default) (color 0 0 0 0))
+  )
+  (bus (pts (xy 35.56 33.02) (xy 46.99 33.02))
+    (stroke (width 0) (type default) (color 0 0 0 0))
+  )
   (wire (pts (xy 96.52 161.29) (xy 115.57 161.29))
     (stroke (width 0) (type default) (color 0 0 0 0))
@@
     (stroke (width 0) (type default) (color 0 0 0 0))
   )
+  (bus (pts (xy 35.56 35.56) (xy 46.99 35.56))
+    (stroke (width 0) (type default) (color 0 0 0 0))
+  )
   (wire (pts (xy 96.52 154.94) (xy 115.57 154.94))
     (stroke (width 0) (type default) (color 0 0 0 0))
@@
     (stroke (width 0) (type default) (color 0 0 0 0))
   )
+  (bus (pts (xy 35.56 27.94) (xy 46.99 27.94))
+    (stroke (width 0) (type default) (color 0 0 0 0))
+  )
   (wire (pts (xy 96.52 115.57) (xy 115.57 115.57))
     (stroke (width 0) (type default) (color 0 0 0 0))
@@
   (wire (pts (xy 96.52 133.35) (xy 115.57 133.35))
     (stroke (width 0) (type default) (color 0 0 0 0))
+  )
+  (text "(notes) POWER SUPPLY\n\n3.3V --> 1.5A\n1.8V --> 0.6A\n1.5V --> 1.2A\n1.0V --> 2.1A"
+    (at 80.01 34.29 0)
+    (effects (font (size 1.27 1.27) italic) (justify right bottom))
+  )
+  (global_label "1.8V" (shape input) (at 46.99 30.48 0) (fields_autoplaced)
+    (effects (font (size 1.27 1.27)) (justify left))
+    (property "Intersheet References" "${INTERSHEET_REFS}" (id 0) (at 53.5155 30.4006 0)
+      (effects (font (size 1.27 1.27)) (justify left) hide)
+    )
+  )
+  (global_label "1.5V" (shape input) (at 46.99 33.02 0) (fields_autoplaced)
+    (effects (font (size 1.27 1.27)) (justify left))
+    (property "Intersheet References" "${INTERSHEET_REFS}" (id 0) (at 53.5155 32.9406 0)
+      (effects (font (size 1.27 1.27)) (justify left) hide)
+    )
+  )
+  (global_label "GND" (shape input) (at 46.99 38.1 0) (fields_autoplaced)
+    (effects (font (size 1.27 1.27)) (justify left))
+    (property "Intersheet References" "${INTERSHEET_REFS}" (id 0) (at 53.2736 38.0206 0)
+      (effects (font (size 1.27 1.27)) (justify left) hide)
+    )
+  )
+  (global_label "5V" (shape input) (at 46.99 25.4 0) (fields_autoplaced)
+    (effects (font (size 1.27 1.27)) (justify left))
+    (property "Intersheet References" "${INTERSHEET_REFS}" (id 0) (at 51.7012 25.3206 0)
+      (effects (font (size 1.27 1.27)) (justify left) hide)
+    )
+  )
+  (global_label "3.3V" (shape input) (at 46.99 27.94 0) (fields_autoplaced)
+    (effects (font (size 1.27 1.27)) (justify left))
+    (property "Intersheet References" "${INTERSHEET_REFS}" (id 0) (at 53.5155 27.8606 0)
+      (effects (font (size 1.27 1.27)) (justify left) hide)
+    )
+  )
+  (global_label "1.0V" (shape input) (at 46.99 35.56 0) (fields_autoplaced)
+    (effects (font (size 1.27 1.27)) (justify left))
+    (property "Intersheet References" "${INTERSHEET_REFS}" (id 0) (at 53.5155 35.4806 0)
+      (effects (font (size 1.27 1.27)) (justify left) hide)
+    )
+  )
+  (symbol (lib_id "Connector:Conn_01x06_Male") (at 30.48 30.48 0) (unit 1)
+    (in_bom yes) (on_board yes) (fields_autoplaced)
+    (property "Reference" "J?" (id 0) (at 31.115 20.32 0))
+    (property "Value" "POWER_SOURCE" (id 1) (at 31.115 22.86 0))
+    (property "Footprint" "Connector_PinHeader_2.54mm:PinHeader_1x06_P2.54mm_Vertical" (id 2) (at 30.48 30.48 0)
+      (effects (font (size 1.27 1.27)) hide)
+    )
+    (property "Datasheet" "~" (id 3) (at 30.48 30.48 0)
+      (effects (font (size 1.27 1.27)) hide)
+    )
+    (pin "1")
+    (pin "2")
+    (pin "3")
+    (pin "4")
+    (pin "5")
+    (pin "6")
   )
   (sheet (at 58.42 88.9) (size 38.1 81.28) (fields_autoplaced)
@@
     )
   )
-  (sheet (at 66.04 59.69) (size 25.4 8.89) (fields_autoplaced)
-    (stroke (width 0.1524) (type solid) (color 0 0 0 0))
-    (fill (color 0 0 0 0.0000))
-    (property "Sheet name" "POWER_SUPPLY" (id 0) (at 66.04 58.9784 0)
-      (effects (font (size 1.27 1.27)) (justify left bottom))
-    )
-    (property "Sheet file" "POWER_sch.kicad_sch" (id 1) (at 66.04 69.1646 0)
-      (effects (font (size 1.27 1.27)) (justify left top))
-    )
-  )
   (sheet_instances
     (path "/" (page "1"))
     (path "/40db1252-e8c0-4f72-a749-2ec7d29f42a9" (page "2"))
     (path "/54d0b93a-ed98-4e03-bfbf-76e3073701f9" (page "3"))
-    (path "/5c445b91-08f8-474d-8e69-7b48e2ef0283" (page "4"))
   )
   (symbol_instances
@@
       (reference "IC2") (unit 1) (value "MT41J128M16JT-125_K") (footprint "DDR:BGA96C80P9X16_800X1400X120")
     )
-    (path "/5c445b91-08f8-474d-8e69-7b48e2ef0283/b2507905-38a8-4be8-9259-9da0c393189c"
-      (reference "J1") (unit 1) (value "POWER_SOURCE") (footprint "Connector_PinHeader_2.54mm:PinHeader_1x06_P2.54mm_Vertical")
-    )
-  )
+    (path "/4e6ad2f4-4822-4162-ba24-28e1c73f86e8"
+      (reference "J?") (unit 1) (value "POWER_SOURCE") (footprint "Connector_PinHeader_2.54mm:PinHeader_1x06_P2.54mm_Vertical")
+    )
+  )
