File: zynq/zynq.kicad_pcb (KiCad board)
At the start: 2 copper layers, 1 part, among them IC1 XC7Z010-1CLG400C

Commit message: .
Parts:
- added IC2: MT41J128M16JT-125_K, DDR:BGA96C80P9X16_800X1400X120, F.Cu at (89.0, 71.1)
- added J1: POWER_SOURCE, Connector_PinHeader_2.54mm:PinHeader_1x06_P2.54mm_Vertical, F.Cu at (147.3, 85.1)
- IC1: value XC7Z010-1CLG400C -> ~
- moved IC1 42.7 mm to (109.1, 71.1)
Connections:
- IC1 pad D4: unconnected-(IC1-PadD4) -> /CPU/DDR3_A13
- IC1 pad E4: unconnected-(IC1-PadE4) -> /CPU/DDR3_A12
- IC1 pad F4: unconnected-(IC1-PadF4) -> /CPU/DDR3_A14
- IC1 pad F5: unconnected-(IC1-PadF5) -> /CPU/DDR3_A10
- IC1 pad G4: unconnected-(IC1-PadG4) -> /CPU/DDR3_A11
- IC1 pad J4: unconnected-(IC1-PadJ4) -> /CPU/DDR3_A9
- IC1 pad K1: unconnected-(IC1-PadK1) -> /CPU/DDR3_A8
- IC1 pad K2: unconnected-(IC1-PadK2) -> /CPU/DDR3_A1
- IC1 pad K3: unconnected-(IC1-PadK3) -> /CPU/DDR3_A3
- IC1 pad K4: unconnected-(IC1-PadK4) -> /CPU/DDR3_A7
- IC1 pad L1: unconnected-(IC1-PadL1) -> /CPU/DDR3_A5
- IC1 pad L4: unconnected-(IC1-PadL4) -> /CPU/DDR3_A6
- IC1 pad M3: unconnected-(IC1-PadM3) -> /CPU/DDR3_A2
- IC1 pad M4: unconnected-(IC1-PadM4) -> /CPU/DDR3_A4
- IC1 pad N2: unconnected-(IC1-PadN2) -> /CPU/DDR3_A0
Routing:
- net /CPU/DDR3_A11: track 0.00 -> 11.7 mm
Other:
- board outline added: 88.9 x 53.3 mm

Commit message: .
Parts:
- moved IC2 2.56 mm to (88.1, 68.7)
Connections:
- net /DRAM/GND renamed /DDR3/GND
- net /DRAM/VCC1V5 renamed /DDR3/VCC1V5
- IC1 pad A2: unconnected-(IC1-PadA2) -> /CPU/DDR3_D13
- IC1 pad A4: unconnected-(IC1-PadA4) -> /CPU/DDR3_D15
- IC1 pad B3: unconnected-(IC1-PadB3) -> /CPU/DDR3_D12
- IC1 pad C1: unconnected-(IC1-PadC1) -> /CPU/DDR3_D10
- IC1 pad C3: unconnected-(IC1-PadC3) -> /CPU/DDR3_D11
- IC1 pad D1: unconnected-(IC1-PadD1) -> /CPU/DDR3_D14
- IC1 pad D3: unconnected-(IC1-PadD3) -> /CPU/DDR3_D8
- IC1 pad E1: unconnected-(IC1-PadE1) -> /CPU/DDR3_D9
- IC1 pad E2: unconnected-(IC1-PadE2) -> /CPU/DDR3_D2
- IC1 pad E3: unconnected-(IC1-PadE3) -> /CPU/DDR3_D0
- IC1 pad G3: unconnected-(IC1-PadG3) -> /CPU/DDR3_D3
- IC1 pad H1: unconnected-(IC1-PadH1) -> /CPU/DDR3_D7
- IC1 pad H2: unconnected-(IC1-PadH2) -> /CPU/DDR3_D1
- IC1 pad H3: unconnected-(IC1-PadH3) -> /CPU/DDR3_D5
- IC1 pad J1: unconnected-(IC1-PadJ1) -> /CPU/DDR3_D4
- IC1 pad J3: unconnected-(IC1-PadJ3) -> /CPU/DDR3_D6
- IC1 pad J5: unconnected-(IC1-PadJ5) -> /CPU/DDR3_BA2
- IC1 pad L2: unconnected-(IC1-PadL2) -> /CPU/DDR3_CK_P
- IC1 pad L5: unconnected-(IC1-PadL5) -> /CPU/DDR3_BA0
- IC1 pad M2: unconnected-(IC1-PadM2) -> /CPU/DDR3_CK_N
- IC1 pad N3: unconnected-(IC1-PadN3) -> /CPU/DDR3_CKE0
- IC1 pad R4: unconnected-(IC1-PadR4) -> /CPU/DDR3_BA1
- IC2 pad A2: unconnected-(IC2-PadA2) -> /CPU/DDR3_D13
- IC2 pad A3: unconnected-(IC2-PadA3) -> /CPU/DDR3_D15
- IC2 pad A7: unconnected-(IC2-PadA7) -> /CPU/DDR3_D12
- IC2 pad B8: unconnected-(IC2-PadB8) -> /CPU/DDR3_D14
- IC2 pad C2: unconnected-(IC2-PadC2) -> /CPU/DDR3_D11
- IC2 pad C3: unconnected-(IC2-PadC3) -> /CPU/DDR3_D9
- IC2 pad C8: unconnected-(IC2-PadC8) -> /CPU/DDR3_D10
- IC2 pad D7: unconnected-(IC2-PadD7) -> /CPU/DDR3_D8
- IC2 pad E3: unconnected-(IC2-PadE3) -> /CPU/DDR3_D0
- IC2 pad F2: unconnected-(IC2-PadF2) -> /CPU/DDR3_D2
- IC2 pad F7: unconnected-(IC2-PadF7) -> /CPU/DDR3_D1
- IC2 pad F8: unconnected-(IC2-PadF8) -> /CPU/DDR3_D3
- IC2 pad G2: unconnected-(IC2-PadG2) -> /CPU/DDR3_D6
- IC2 pad H3: unconnected-(IC2-PadH3) -> /CPU/DDR3_D4
- IC2 pad H7: unconnected-(IC2-PadH7) -> /CPU/DDR3_D7
- IC2 pad H8: unconnected-(IC2-PadH8) -> /CPU/DDR3_D5
- IC2 pad J7: unconnected-(IC2-PadJ7) -> /CPU/DDR3_CK_P
- IC2 pad K7: unconnected-(IC2-PadK7) -> /CPU/DDR3_CK_N
- IC2 pad K9: unconnected-(IC2-PadK9) -> /CPU/DDR3_CKE0
- IC2 pad M2: unconnected-(IC2-PadM2) -> /CPU/DDR3_BA0
- IC2 pad M3: unconnected-(IC2-PadM3) -> /CPU/DDR3_BA2
- IC2 pad N8: unconnected-(IC2-PadN8) -> /CPU/DDR3_BA1
Routing:
- net /CPU/DDR3_A11: track 11.7 -> 0.00 mm

Commit message: .
Parts:
- moved IC2 2.63 mm to (90.0, 67.0)
Changed lines of the file:
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@@
   (net 465 "/CPU/DDR3_A0")
   (footprint "DDR:BGA96C80P9X16_800X1400X120" (layer "F.Cu")
-    (at 88.09 68.74 90)
+    (at 90.03 66.96 90)
     (descr "96-Ball FBGA ??x16 (JT)%0 ")
     (tags "Integrated Circuit")

Commit message: .
Parts:
- moved IC2 1.47 mm to (88.9, 68.0)
Routing:
- net /CPU/DDR3_A0: track 0.00 -> 17.2 mm
- net /CPU/DDR3_A2: track 0.00 -> 15.8 mm
- net /CPU/DDR3_A3: track 0.00 -> 13.5 mm
- net /CPU/DDR3_A13: track 0.00 -> 11.9 mm
- net /CPU/DDR3_A9: track 0.00 -> 10.3 mm
- net /CPU/DDR3_A7: track 0.00 -> 10.3 mm
- net /CPU/DDR3_A5: track 0.00 -> 10.2 mm
Other:
- copper layers 2 -> 6
Changed lines of the file:
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@@
 (kicad_pcb (version 20211014) (generator pcbnew)
   (general
-    (thickness 1.6)
+    (thickness 7.78)
   )
   (paper "A4")
   (layers
     (0 "F.Cu" signal)
+    (1 "In1.Cu" signal)
+    (2 "In2.Cu" signal)
+    (3 "In3.Cu" signal)
+    (4 "In4.Cu" signal)
     (31 "B.Cu" signal)
     (32 "B.Adhes" user "B.Adhesive")
@@
       (layer "F.Cu" (type "copper") (thickness 0.035))
       (layer "dielectric 1" (type "core") (thickness 1.51) (material "FR4") (epsilon_r 4.5) (loss_tangent 0.02))
+      (layer "In1.Cu" (type "copper") (thickness 0.035))
+      (layer "dielectric 2" (type "prepreg") (thickness 1.51) (material "FR4") (epsilon_r 4.5) (loss_tangent 0.02))
+      (layer "In2.Cu" (type "copper") (thickness 0.035))
+      (layer "dielectric 3" (type "core") (thickness 1.51) (material "FR4") (epsilon_r 4.5) (loss_tangent 0.02))
+      (layer "In3.Cu" (type "copper") (thickness 0.035))
+      (layer "dielectric 4" (type "prepreg") (thickness 1.51) (material "FR4") (epsilon_r 4.5) (loss_tangent 0.02))
+      (layer "In4.Cu" (type "copper") (thickness 0.035))
+      (layer "dielectric 5" (type "core") (thickness 1.51) (material "FR4") (epsilon_r 4.5) (loss_tangent 0.02))
       (layer "B.Cu" (type "copper") (thickness 0.035))
       (layer "B.Mask" (type "Bottom Solder Mask") (thickness 0.01))
@@
   (net 465 "/CPU/DDR3_A0")
   (footprint "DDR:BGA96C80P9X16_800X1400X120" (layer "F.Cu")
-    (at 90.03 66.96 90)
+    (at 88.94 67.95 90)
     (descr "96-Ball FBGA ??x16 (JT)%0 ")
     (tags "Integrated Circuit")
@@
   )
   (gr_rect (start 66.04 50.8) (end 154.94 104.14) (layer "Edge.Cuts") (width 0.1) (fill none))
+  (segment (start 103.36 68.77) (end 103.46 68.67) (width 0.1) (layer "F.Cu") (net 64))
+  (segment (start 101.33 68.815716) (end 101.33 68.77) (width 0.1) (layer "F.Cu") (net 64))
+  (segment (start 101.33 68.77) (end 103.36 68.77) (width 0.1) (layer "F.Cu") (net 64))
+  (segment (start 103.46 68.67) (end 103.46 66.38) (width 0.1) (layer "F.Cu") (net 64))
+  (segment (start 94.94 69.55) (end 94.94 69.46) (width 0.1) (layer "F.Cu") (net 64))
+  (segment (start 94.94 69.46) (end 95.26 69.14) (width 0.1) (layer "F.Cu") (net 64))
+  (segment (start 103.46 66.38) (end 103.9 65.94) (width 0.1) (layer "F.Cu") (net 64))
+  (segment (start 95.26 69.14) (end 101.005716 69.14) (width 0.1) (layer "F.Cu") (net 64))
+  (segment (start 101.005716 69.14) (end 101.33 68.815716) (width 0.1) (layer "F.Cu") (net 64))
+  (segment (start 94.14 69.55) (end 94.585489 69.995489) (width 0.1) (layer "F.Cu") (net 164))
+  (segment (start 103.46 69.5) (end 103.9 69.94) (width 0.1) (layer "F.Cu") (net 164))
+  (segment (start 101.445716 69.5) (end 103.46 69.5) (width 0.1) (layer "F.Cu") (net 164))
+  (segment (start 100.950227 69.995489) (end 101.445716 69.5) (width 0.1) (layer "F.Cu") (net 164))
+  (segment (start 94.585489 69.995489) (end 100.950227 69.995489) (width 0.1) (layer "F.Cu") (net 164))
+  (segment (start 101.150489 72.195227) (end 101.355227 71.990489) (width 0.1) (layer "F.Cu") (net 182))
+  (segment (start 101.355227 71.990489) (end 102.444773 71.990489) (width 0.1) (layer "F.Cu") (net 182))
+  (segment (start 101.150489 72.28) (end 101.150489 72.195227) (width 0.1) (layer "F.Cu") (net 182))
+  (segment (start 102.750489 71.684773) (end 102.750489 71.089511) (width 0.1) (layer "F.Cu") (net 182))
+  (segment (start 102.750489 71.089511) (end 103.1 70.74) (width 0.1) (layer "F.Cu") (net 182))
+  (segment (start 92.185489 71.385489) (end 93.08 72.28) (width 0.1) (layer "F.Cu") (net 182))
+  (segment (start 93.08 72.28) (end 101.150489 72.28) (width 0.1) (layer "F.Cu") (net 182))
+  (segment (start 92.54 70.35) (end 92.185489 70.704511) (width 0.1) (layer "F.Cu") (net 182))
+  (segment (start 92.185489 70.704511) (end 92.185489 71.385489) (width 0.1) (layer "F.Cu") (net 182))
+  (segment (start 102.444773 71.990489) (end 102.750489 71.684773) (width 0.1) (layer "F.Cu") (net 182))
+  (segment (start 96.144511 70.795489) (end 96.549511 70.390489) (width 0.1) (layer "F.Cu") (net 183))
+  (segment (start 96.549511 70.390489) (end 103.550489 70.390489) (width 0.1) (layer "F.Cu") (net 183))
+  (segment (start 94.585489 70.795489) (end 96.144511 70.795489) (width 0.1) (layer "F.Cu") (net 183))
+  (segment (start 94.14 70.35) (end 94.585489 70.795489) (width 0.1) (layer "F.Cu") (net 183))
+  (segment (start 103.550489 70.390489) (end 103.9 70.74) (width 0.1) (layer "F.Cu") (net 183))
+  (segment (start 92.985489 70.704511) (end 92.985489 71.345489) (width 0.1) (layer "F.Cu") (net 200))
+  (segment (start 93.72048 72.08048) (end 100.95952 72.08048) (width 0.1) (layer "F.Cu") (net 200))
+  (segment (start 92.985489 71.345489) (end 93.72048 72.08048) (width 0.1) (layer "F.Cu") (net 200))
+  (segment (start 100.95952 72.08048) (end 101.5 71.54) (width 0.1) (layer "F.Cu") (net 200))
+  (segment (start 93.34 70.35) (end 92.985489 70.704511) (width 0.1) (layer "F.Cu") (net 200))
+  (segment (start 91.765489 69.904511) (end 91.71 69.96) (width 0.1) (layer "F.Cu") (net 464))
+  (segment (start 93.96 72.54) (end 94.109511 72.689511) (width 0.1) (layer "F.Cu") (net 464))
+  (segment (start 91.71 69.96) (end 91.628645 69.96) (width 0.1) (layer "F.Cu") (net 464))
+  (segment (start 93.34 69.55) (end 92.985489 69.904511) (width 0.1) (layer "F.Cu") (net 464))
+  (segment (start 102.750489 72.689511) (end 103.1 72.34) (width 0.1) (layer "F.Cu") (net 464))
+  (segment (start 91.628645 69.96) (end 91.385489 70.203156) (width 0.1) (layer "F.Cu") (net 464))
+  (segment (start 91.385489 70.203156) (end 91.385489 71.315489) (width 0.1) (layer "F.Cu") (net 464))
+  (segment (start 94.109511 72.689511) (end 102.750489 72.689511) (width 0.1) (layer "F.Cu") (net 464))
+  (segment (start 92.61 72.54) (end 93.96 72.54) (width 0.1) (layer "F.Cu") (net 464))
+  (segment (start 91.385489 71.315489) (end 92.61 72.54) (width 0.1) (layer "F.Cu") (net 464))
+  (segment (start 92.985489 69.904511) (end 91.765489 69.904511) (width 0.1) (layer "F.Cu") (net 464))
+  (segment (start 92.54 69.55) (end 92.06 69.07) (width 0.1) (layer "F.Cu") (net 465))
+  (segment (start 90.585489 71.665489) (end 92.45 73.53) (width 0.1) (layer "F.Cu") (net 465))
+  (segment (start 90.91 69.07) (end 90.585489 69.394511) (width 0.1) (layer "F.Cu") (net 465))
+  (segment (start 92.06 69.07) (end 90.91 69.07) (width 0.1) (layer "F.Cu") (net 465))
+  (segment (start 101.91 73.53) (end 102.3 73.14) (width 0.1) (layer "F.Cu") (net 465))
+  (segment (start 90.585489 69.394511) (end 90.585489 71.665489) (width 0.1) (layer "F.Cu") (net 465))
+  (segment (start 92.45 73.53) (end 101.91 73.53) (width 0.1) (layer "F.Cu") (net 465))
 )
